Commit message: Sim no_link bug fixed

File: sim_catkin_ws/src/ardupilot_sitl_gazebo_plugin/ardupilot_sitl_gazebo_plugin/urdf/hedwig_quad.xacro (robot description, xacro)
@@ -168,8 +168,8 @@
     <origin xyz="0.13 0.0 0.07" rpy="0 0 0"/>
   </xacro:lidar_sensor>
-  <!-- Downward facing camera -->
+  <!-- Downward facing cameras -->
   <xacro:include filename="$(find ardupilot_sitl_gazebo_plugin)/urdf/sensors/generic_camera.urdf.xacro" />
   <xacro:generic_camera
-    name="erlecopter/left"
+    name="erlecopter/bottom"
     parent="base_link"
     ros_topic="image_raw"
@@ -177,14 +177,28 @@
     update_rate="60"
     res_x="640"
-    res_y="480"
-    image_format="R8G8B8"
-    hfov="45"
+    res_y="360"
+    image_format="R8G8B8"
+    hfov="81"
     framename="erlecopter_bottomcam">
-    <origin xyz="0.14 0.2 -0.02" rpy="0 ${45*M_PI/180} 0"/>
+    <origin xyz="0.00 0.2 -0.02" rpy="0 ${45*M_PI/180} 0"/>
   </xacro:generic_camera>
-  <!-- Front facing camera -->
   <xacro:include filename="$(find ardupilot_sitl_gazebo_plugin)/urdf/sensors/generic_camera.urdf.xacro" />
   <xacro:generic_camera
-    name="erlecopter/right"
+    name="erlecopter/front"
+    parent="base_link"
+    ros_topic="image_front_raw"
+    cam_info_topic="camera_front_info"
+    update_rate="25"
+    res_x="640"
+    res_y="360"
+    image_format="R8G8B8"
+    hfov="81"
+    framename="erlecopter_frontcam">
+    <origin xyz="0.00 -0.2 -0.02" rpy="0 ${45*M_PI/180} 0"/>
+  </xacro:generic_camera>
+  <!-- Downward facing cameras
+  <xacro:include filename="$(find ardupilot_sitl_gazebo_plugin)/urdf/sensors/generic_camera.urdf.xacro" />
+  <xacro:generic_camera
+   name="erlecopter/bottom"
     parent="base_link"
     ros_topic="image_raw"
@@ -192,10 +206,24 @@
     update_rate="60"
     res_x="640"
-    res_y="480"
-    image_format="R8G8B8"
-    hfov="45"
+    res_y="360"
+    image_format="R8G8B8"
+    hfov="81"
+    framename="erlecopter_bottomcam">
+    <origin xyz="0.14 0.2 -0.02" rpy="0 ${45*M_PI/180} 0"/>
+  </xacro:generic_camera>
+  <xacro:include filename="$(find ardupilot_sitl_gazebo_plugin)/urdf/sensors/generic_camera.urdf.xacro" />
+  <xacro:generic_camera
+    name="erlecopter/front"
+    parent="base_link"
+    ros_topic="image_front_raw"
+    cam_info_topic="camera_front_info"
+    update_rate="25"
+    res_x="640"
+    res_y="360"
+    image_format="R8G8B8"
+    hfov="81"
     framename="erlecopter_frontcam">
     <origin xyz="0.14 -0.2 -0.02" rpy="0 ${45*M_PI/180} 0"/>
-  </xacro:generic_camera>
+  </xacro:generic_camera> -->
   <!-- Instantiate rotors -->
   <xacro:vertical_rotor

Commit message: Add Stereo Altitude Ground truth based on sonar sensor

File: sim_catkin_ws/src/ardupilot_sitl_gazebo_plugin/ardupilot_sitl_gazebo_plugin/urdf/hedwig_quad.xacro (robot description, xacro)
@@ -139,19 +139,18 @@
     <origin xyz="0.12 0.0 0.0" rpy="0 ${90*M_PI/180} 0"/>
   </xacro:sonar_sensor>
-    <!-- Frontal range sensor -->
-<!--  <xacro:sonar_sensor
-    name="sonar2"
-    parent="base_link"
-    ros_topic="sonar_front"
+    <!-- Stereo Altitude Ground Truth -->
+  <xacro:sonar_sensor
+    name="sonar3"
+    parent="base_link"
+    ros_topic="stereo_altitude_gt"
     update_rate="10"
     min_range="0.01"
-    max_range="50.0"
+    max_range="150.0"
     field_of_view="${1*M_PI/180}"
     ray_count="1"
     sensor_mesh="lidar_lite_v2_withRay/meshes/lidar_lite_v2_withRay.dae">
-    <origin xyz="0.13 0.0 0.02" rpy="0 0 0"/>
+    <origin xyz="0.00 0.00 -0.02" rpy="0 ${45*M_PI/180} 0"/>
   </xacro:sonar_sensor>
--->
-  <xacro:include filename="$(find ardupilot_sitl_gazebo_plugin)/urdf/sensors/lidar_sensor.urdf.xacro" />
+ <!-- <xacro:include filename="$(find ardupilot_sitl_gazebo_plugin)/urdf/sensors/lidar_sensor.urdf.xacro" />
    <xacro:lidar_sensor
     name="sonar2"
@@ -167,5 +166,5 @@
     sensor_mesh="lidar_lite_v2_withRay/meshes/lidar_lite_v2_withRay.dae">
     <origin xyz="0.13 0.0 0.07" rpy="0 0 0"/>
-  </xacro:lidar_sensor>
+  </xacro:lidar_sensor>-->
   <!-- Downward facing cameras -->
   <xacro:include filename="$(find ardupilot_sitl_gazebo_plugin)/urdf/sensors/generic_camera.urdf.xacro" />
